File: psu/psu.kicad_sch (KiCad schematic)
At the start: 35 parts, among them J1 220VAC, J2 Vout conn, J3 OLED Pins, Q1 tip35c, Q2 BD139, Q3 BC184C, Q4 NPN, SW1 Main, T1 220/24, U1 TL431LP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

Commit message: Fixed a floating emitter
Connections:
- net DCOUT-: now also Q4.3 (E)
Changed lines of the file:
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@@
+	)
+	(junction
+		(at 210.82 146.05)
+		(diameter 0)
+		(color 0 0 0 0)
 	)
 	(junction
@@
 	(wire
 		(pts
+			(xy 240.03 146.05) (xy 210.82 146.05)
+		)
+		(stroke
+			(width 0)
+			(type default)
+		)
+	)
+	(wire
+		(pts
 			(xy 101.6 38.1) (xy 101.6 62.23)
 		)
@@
 		)
 		(stroke
+			(width 0)
+			(type default)
+		)
+	)
+	(wire
+		(pts
+			(xy 240.03 129.54) (xy 240.03 146.05)
+		)
+		(stroke
