File: CAD/psu.kicad_pcb (KiCad board)
At the start: 2 copper layers, 85.5 x 107 mm, 34 parts, among them J1 220VAC, J2 Vout conn, J3 OLED Pins, J4 GND/-, Q1 tip35c, Q2 BD139, Q3 BC184C, Q4 BC547, SW1 Main, T1 220/24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

Commit message: Major PCB redesign, transformr goes on a different PCB, while the LEDs and potentiometers go to the front panel, as well as the fuse and main switch."
Parts:
- removed F1: 350mA, Fuse:Fuseholder_Clip-5x20mm_Eaton_1A5601-01_Inline_P20.80x6.76mm_D1.70mm_Horizontal
- removed J1: 220VAC, Connector_Samtec_HPM_THT:Samtec_HPM-03-05-x-S_Straight_1x03_Pitch5.08mm
- removed SW1: Main, Button_Switch_THT:SW_DIP_SPSTx01_Piano_10.8x4.1mm_W7.62mm_P2.54mm
- added C1: 4700uF 40V, Capacitor_THT:CP_Radial_D18.0mm_P7.50mm, F.Cu at (100.0, 44.0)
- added C2: 470uF 40v, Capacitor_THT:CP_Radial_D18.0mm_P7.50mm, F.Cu at (83.5, 60.5)
- T1: footprint Transformer_THT:Transformer_Zeming_ZMPT101K -> Connector_PinHeader_2.54mm:PinHeader_1x02_P2.54mm_Vertical
- moved T1 15.3 mm to (103.0, 116.7), turned to 0 degrees
Routing:
- net Net-(T1-AA): track 148.3 -> 2.80 mm
- net Net-(J1-N): track 73.3 -> 11.4 mm
- net Net-(T1-SA): track 61.0 -> 25.3 mm
- net Net-(T1-SB): track 46.7 -> 17.6 mm
- net /DCOUT: track 263.1 -> 283.8 mm
- net GND: track 168.0 -> 153.2 mm
- net /DCOUT-: track 261.4 -> 275.7 mm
- net Net-(SW1-B): track 13.6 -> 0.00 mm
- net Vout: track 93.8 -> 106.2 mm, vias 0 -> 1
- net Net-(J1-L): track 8.77 -> 0.00 mm
Other:
- board text removed: "L"
- board text removed: "N"
