File: CAD/psu.kicad_sch (KiCad schematic)
At the start: 35 parts, among them J1 220VAC, J2 Vout conn, J3 OLED Pins, Q1 tip35c, Q2 BD139, Q3 BC184C, Q4 NPN, SW1 Main, T1 220/24, U1 TL431LP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

Commit message: PCB designed, and working on the readme
Parts:
- removed 0.5/5W: R, Resistor_THT:R_Axial_DIN0922_L20.0mm_D9.0mm_P30.48mm_Horizontal, symbol Device:R
- added J4: GND/-, Connector:Banana_Jack_1Pin, symbol Connector:Conn_01x01_Socket
- added R7: 0R5/5W, Resistor_THT:R_Axial_Power_L20.0mm_W6.4mm_P25.40mm, symbol Device:R
- BZ1: footprint (none) -> Buzzer_Beeper:Buzzer_15x7.5RM7.6
- C3: footprint (none) -> Capacitor_THT:C_Disc_D10.0mm_W2.5mm_P5.00mm
- C4: footprint (none) -> Capacitor_THT:CP_Radial_D10.0mm_P2.50mm
- D1: footprint Diode_SMD:Diode_Bridge_Diotec_ABS -> Diode_THT:Diode_Bridge_Vishay_GBL
- D2, D4: footprint (none) -> LED_THT:LED_D3.0mm
- D3: footprint (none) -> Diode_THT:D_DO-41_SOD81_P10.16mm_Horizontal
- F1: footprint (none) -> Fuse:Fuseholder_Clip-5x20mm_Eaton_1A5601-01_Inline_P20.80x6.76mm_D1.70mm_Horizontal
- J1: footprint (none) -> Connector_Samtec_HPM_THT:Samtec_HPM-03-05-x-S_Straight_1x03_Pitch5.08mm
- J2: footprint (none) -> Connector:Banana_Jack_1Pin
- J3: footprint (none) -> Connector_PinSocket_2.54mm:PinSocket_1x04_P2.54mm_Vertical
- K1: footprint (none) -> Relay_THT:Relay_SPST_Omron_G5NB
- Q1: footprint (none) -> Package_TO_SOT_THT:TO-247-3_Vertical
- Q2: footprint (none) -> Package_TO_SOT_THT:TO-126-3_Vertical
- Q3: footprint (none) -> Package_TO_SOT_THT:TO-92
- Q4: value NPN -> BC547; footprint (none) -> Package_TO_SOT_THT:TO-92
- R1, R2, R3, R4, R5: footprint (none) -> Resistor_THT:R_Axial_DIN0207_L6.3mm_D2.5mm_P2.54mm_Vertical
- R6: value R -> 220; footprint (none) -> Resistor_THT:R_Axial_DIN0207_L6.3mm_D2.5mm_P2.54mm_Vertical
- RV1, RV2: footprint (none) -> Potentiometer_THT:Potentiometer_ACP_CA14-H2,5_Horizontal
- RV3, RV4: footprint (none) -> Potentiometer_THT:Potentiometer_Runtron_RM-063_Horizontal
- SW1: footprint (none) -> Button_Switch_THT:SW_DIP_SPSTx01_Piano_10.8x4.1mm_W7.62mm_P2.54mm
- T1: footprint (none) -> Transformer_THT:Transformer_Zeming_ZMPT101K
Connections:
- net DCOUT-: now also R7.1
- net GND: now also J4.1 (Pin_1), R7.2
- no-connect marks 0 -> 20

Commit message: Pushing some minor footprint changes in the SCH.
Parts:
- C1, C2: footprint (none) -> Capacitor_THT:CP_Radial_D18.0mm_P7.50mm
- T1: footprint Transformer_THT:Transformer_Zeming_ZMPT101K -> Connector_PinHeader_2.54mm:PinHeader_1x02_P2.54mm_Vertical
Changed lines of the file:
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@@
 			)
 		)
-		(property "Footprint" ""
+		(property "Footprint" "Capacitor_THT:CP_Radial_D18.0mm_P7.50mm"
 			(at 195.2752 46.99 0)
 			(hide yes)
@@
 			)
 		)
-		(property "Footprint" ""
+		(property "Footprint" "Capacitor_THT:CP_Radial_D18.0mm_P7.50mm"
 			(at 102.5652 38.1 0)
 			(hide yes)
@@
 			)
 		)
-		(property "Footprint" "Transformer_THT:Transformer_Zeming_ZMPT101K"
+		(property "Footprint" "Connector_PinHeader_2.54mm:PinHeader_1x02_P2.54mm_Vertical"
 			(at 71.12 26.67 0)
 			(hide yes)
